File: audio chain.kicad_pcb (KiCad board)
At the start: 2 copper layers, 26 parts, among them IC2 LM2902AWYDT, IC4 LM2902AWYDT

Commit message: updates
Connections:
- IC2 pad 8: Net-(C1-Pad1) -> Net-(C2-Pad1)
- R1 pad 1: Net-(IC2-Pad2) -> Net-(IC1-Pad2)
- R1 pad 2: Net-(IC2-Pad1) -> Net-(IC1-Pad1)
- R10 pad 1: Net-(IC4-Pad6) -> Net-(IC2-Pad6)
- R11 pad 2: Net-(IC2-Pad13) -> Net-(IC1-Pad13)
- R12 pad 1: Net-(IC2-Pad9) -> Net-(IC1-Pad9)
- R13 pad 1: Net-(IC2-Pad9) -> Net-(IC1-Pad9)
- R14 pad 2: Net-(IC4-Pad13) -> Net-(IC2-Pad13)
- R15 pad 2: Net-(IC4-Pad13) -> Net-(IC2-Pad13)
- R16 pad 1: Net-(IC4-Pad9) -> Net-(IC2-Pad9)
- R17 pad 1: Net-(IC4-Pad9) -> Net-(IC2-Pad9)
- R18 pad 1: Net-(IC2-Pad13) -> Net-(IC1-Pad13)
- R18 pad 2: Net-(IC2-Pad14) -> Net-(IC1-Pad14)
- R19 pad 1: Net-(IC2-Pad13) -> Net-(IC1-Pad13)
- R19 pad 2: Net-(IC2-Pad14) -> Net-(IC1-Pad14)
- R2 pad 1: Net-(IC2-Pad2) -> Net-(IC1-Pad2)
- R20 pad 1: Net-(IC4-Pad13) -> Net-(IC2-Pad13)
- R20 pad 2: Net-(IC4-Pad14) -> Net-(IC2-Pad14)
- R21 pad 1: Net-(IC4-Pad13) -> Net-(IC2-Pad13)
- R21 pad 2: Net-(IC4-Pad14) -> Net-(IC2-Pad14)
- R3 pad 1: Net-(IC4-Pad2) -> Net-(IC2-Pad2)
- R3 pad 2: Net-(IC4-Pad1) -> Net-(IC2-Pad1)
- R4 pad 1: Net-(IC4-Pad2) -> Net-(IC2-Pad2)
- R5 pad 1: Net-(IC2-Pad6) -> Net-(IC1-Pad6)
- R5 pad 2: Net-(IC2-Pad10) -> Net-(IC1-Pad10)
- R6 pad 1: Net-(IC2-Pad6) -> Net-(IC1-Pad6)
- R8 pad 1: Net-(IC4-Pad6) -> Net-(IC2-Pad6)
- R8 pad 2: Net-(IC4-Pad10) -> Net-(IC2-Pad10)
- R9 pad 2: Net-(IC2-Pad13) -> Net-(IC1-Pad13)
Other:
- net class Default removed
